File: SingleShotICbased.kicad_pcb (KiCad board)
At the start: 2 copper layers, 53.3 x 23.4 mm, 27 parts, among them J1 GM_KP_ALIVE, J2 Conn_01x02_Male, J3 SSR_ANODE, J4 Conn_01x03_Male, U1 NCP781BMN050TAG, U2 NCP781BMN050TAG, U3 TPL5111

Commit message: finished design
Parts:
- added REF**: MountingHole_2.2mm_M2, MountingHole:MountingHole_2.2mm_M2, F.Cu at (116.1, 81.0)
- added REF**: MountingHole_2.2mm_M2, MountingHole:MountingHole_2.2mm_M2, F.Cu at (164.3, 89.9)
- added REF**: MountingHole_2.2mm_M2, MountingHole:MountingHole_2.2mm_M2, F.Cu at (116.1, 84.1)
- added REF**: MountingHole_2.2mm_M2, MountingHole:MountingHole_2.2mm_M2, F.Cu at (116.1, 95.2)
- added REF**: MountingHole_2.2mm_M2, MountingHole:MountingHole_2.2mm_M2, F.Cu at (116.1, 98.0)
- added REF**: MountingHole_2.2mm_M2, MountingHole:MountingHole_2.2mm_M2, F.Cu at (116.1, 100.8)
- added REF**: MountingHole_2.2mm_M2, MountingHole:MountingHole_2.2mm_M2, F.Cu at (164.3, 99.1)
- moved J1 1.78 mm to (160.3, 89.9)
- moved J3 1.78 mm to (160.3, 99.1)
- moved D2 1.52 mm to (161.0, 94.0)
- moved J2 1.14 mm to (120.0, 83.8)
- moved J4 1.14 mm to (120.0, 100.6)
- moved C1 0.51 mm to (131.1, 84.1)
- moved C3 0.51 mm to (145.8, 85.3)
- moved C4 0.51 mm to (138.2, 83.1)
- moved D1 0.51 mm to (157.5, 85.9)
- moved D4 0.51 mm to (157.5, 95.0)
- moved D5 0.51 mm to (139.7, 87.4)
- moved D6 0.51 mm to (127.1, 99.7)
- moved D7 0.51 mm to (127.1, 97.2)
- moved D8 0.51 mm to (124.1, 93.1)
- moved D9 0.51 mm to (124.8, 88.0)
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Routing:
- net /LV_BATT+_RAW: track 6.44 -> 4.79 mm
- net /PLAT_ESTOP: track 7.73 -> 6.08 mm
- net /GRND_ESTP: track 7.73 -> 6.08 mm
- net Net-(D2-Pad1): track 8.59 -> 6.97 mm
- net Net-(D2-Pad2): track 7.75 -> 6.59 mm
- net /TMATICS: track 6.01 -> 5.15 mm
- net Earth: vias 0 -> 23
Other:
- board text added: "GM_KEEP_ ALIVE"
- board text added: "SSR_ANODE"
